File: PTP_Marko_Pticek_Project1.kicad_sch (KiCad schematic)
At the start: 0 parts

Commit message: ispunjena sastavnica
Parts:
- added R1, R2: R_Small, symbol Device:R_Small
Connections:
- new net +3.3V: R2.1
- new net GND: R1.2
- new net u_iz: R1.1, R2.2
Other:
- company: (none) -> TVZ
- title: (none) -> BCD Brojač

Commit message: shema nadodana - ne555
Parts:
- removed R1, R2: R_Small, symbol Device:R_Small
- added C3: 22u, symbol Device:C_Polarized
- added C4: 1u, symbol Device:C
- added C6: 220U, symbol Device:C_Polarized
- added C7: 10u, symbol Device:C
- added C8: 100n, symbol Device:C
- added D1: 11DQ06, symbol Device:D_Schottky_Filled
- added D2, D3, D4, D5: LED, symbol Device:LED
- added J1: Screw_Terminal_01x02, symbol Connector:Screw_Terminal_01x02
- added L1: 330u, symbol Device:L
- added R1, R2: 2k, symbol Device:R
- added R3, R4: 47k, symbol Device:R
- added R6, R7, R8, R9: 4k7, symbol Device:R
- added SW1: SW_Push, symbol Switch:SW_Push
- added SW2: ~, symbol Switch:SW_SPDT
- added U2: LM2574N-5, Package_DIP:DIP-8_W7.62mm, symbol Regulator_Switching:LM2574N-5
- added U5: NE555P, Package_DIP:DIP-8_W7.62mm, symbol Timer:NE555P
Connections:
- net GND: now also C3.2, C4.1, C6.2, C7.2, C8.2, D1.2 (A), J1.2 (Pin_2), R6.2, R7.2, R8.2, R9.2, SW1.1, U2.2 (SGND), U2.3 (~{ON}/OFF), U2.4 (PGND), U5.1 (GND)
- new net: D5.1 (K), R9.1
- new net: D1.1 (K), L1.1, U2.7 (OUT)
- new net: D4.1 (K), R8.1
- new net: R2.1, SW1.2
- new net: C4.2, R1.2, R2.2, SW2.3 (A)
- new net: R3.2, R4.1, U5.7 (DIS)
- new net: C7.1, R4.2, U5.2 (TR), U5.6 (THR)
- new net: D2.1 (K), R6.1
- new net: D3.1 (K), R7.1
- new net +5V: C6.1, C8.1, L1.2, R1.1, R3.1, U2.1 (FB), U5.4 (R), U5.8 (VCC)
- new net 555: SW2.2 (C), U5.3 (Q)
- new net Clock: SW2.1 (B)
- new net Q0: D2.2 (A)
- new net Q1: D3.2 (A)
- new net Q2: D4.2 (A)
- new net Q3: D5.2 (A)
- new net VD: C3.1, J1.1 (Pin_1), U2.5 (VIN)
- no-connect marks 0 -> 1

Commit message: VJ3
Parts:
- added U1: 74LVC1G11, SOT_23_6:SOT-23-6, symbol SN74LVC1G11:SN74LVC1G11
- R7: renamed from R1; value 2k -> 10k
- renumbered C3 to C1, C6 to C2, D2 to D1, D3 to D2, D4 to D3, D1 to D4, U2 to U1
Connections:
- net +5V: now also U1.5 (VCC)
- net Clock: now also R7.2, U1.3 (B)
- net GND: now also J1.1 (Pin_2), U1.2 (GND); no longer J1.2 (Pin_2)
- net Q1: now also U1.6 (C)
- net Q3: now also U1.1 (A)
- net VD: now also J1.2 (Pin_1); no longer J1.1 (Pin_1)
- net at C4.2, R2.2, SW2.3 (A): no longer R7.2
- new net RESET: U1.4 (Y)
Other:
- moved on the sheet: C1, C2, D1, D2, D3, D4, D5, J1, L1, R6, R7, R8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

Commit message: vj4-zavrsavanje
Parts:
- removed U5: NE555P, Package_DIP:DIP-8_W7.62mm, symbol Timer:NE555P
- added H1, H2, H3, H4: MountingHole, symbol Mechanical:MountingHole
- added R10, R11, R12, R15, R9: 10k, symbol Device:R
- added R14, R16, R17, R18, R5, R6, R8: 2k, symbol Device:R
- added U2, U3: 4027, symbol 4xxx:4027
- added U4: 74LS47, symbol 74xx:74LS47
- added U5: FYS-3911BUHR-21, Display_7Segment:7SegmentLED_LTS6760_LTS6780, symbol Display_Character:SM420561N
- added U7: NE555P, Package_DIP:DIP-8_W7.62mm, symbol Timer:NE555P
- C1: footprint (none) -> Capacitor_THT:CP_Radial_D5.0mm_P2.00mm; Manufacturer  (none) -> AISHI; Manufacturer Part Number (none) -> EWH1EM220D11OT
- C2: footprint (none) -> Capacitor_THT:CP_Radial_D5.0mm_P2.00mm; Manufacturer  (none) -> SAMWHA; Manufacturer Part Number  (none) -> RD1A227M05011BB
- C3: renamed from C4; footprint (none) -> Capacitor_SMD:C_1206_3216Metric_Pad1.33x1.80mm_HandSolder; Manufacturer (none) -> SAMSUNG; Manufacturer Part Number  (none) -> CL31B105KBHNNNE
- C4: renamed from C8; footprint (none) -> Capacitor_SMD:C_1206_3216Metric_Pad1.33x1.80mm_HandSolder; Manufacturer  (none) -> SAMSUNG; Manufacturer Part Number  (none) -> CL31B104KBCNNNC
- C5: renamed from C7; footprint (none) -> Capacitor_SMD:C_1206_3216Metric_Pad1.33x1.80mm_HandSolder; Manufacturer  (none) -> SAMSUNG; Manufacturer Part Number  (none) -> CL31A106KBHNNNE
- renumbered R2 to R13, R3 to R19, R4 to R20
Connections:
- net +5V: now also R10.1, R11.1, R12.1, R15.2, R9.1, U2.16 (VDD), U3.16 (VDD), U4.16 (VCC), U5.1 (CC), U5.6 (CC), U7.4 (R), U7.8 (VCC)
- net 555: now also U7.3 (Q)
- net Clock: now also U2.3 (C)
- net GND: now also U2.7 (S), U2.8 (VSS), U2.9 (S), U3.7 (S), U3.8 (VSS), U3.9 (S), U4.8 (GND), U7.1 (GND)
- net Q0: now also U2.1 (Q), U2.13 (C), U4.7 (A)
- net Q1: now also U2.15 (Q), U3.3 (C), U4.1 (B)
- net Q2: now also U3.1 (Q), U3.13 (C), U4.2 (C)
- net Q3: now also U3.15 (Q), U4.6 (D)
- net RESET: now also U2.12 (R), U2.4 (R), U3.12 (R), U3.4 (R)
- net at R19.2, R20.1: now also U7.7 (DIS)
- net at C5.1, R20.2: now also U7.2 (TR), U7.6 (THR)
- new net: R12.2, U3.10 (J), U3.11 (K)
- new net: R14.1, U4.10 (d)
- new net: R8.1, U4.11 (c)
- new net: R6.1, U4.12 (b)
- new net: R5.1, U4.13 (a)
- new net: R18.1, U4.14 (g)
- new net: R17.1, U4.15 (f)
- new net: R15.1, U4.3 (LT), U4.4 (BI), U4.5 (RBI)
- new net: R16.1, U4.9 (e)
- new net: R5.2, U5.10 (A)
- new net: R17.2, U5.2 (F)
- new net: R18.2, U5.3 (G)
- new net: R16.2, U5.4 (E)
- new net: R14.2, U5.5 (D)
- new net: R8.2, U5.8 (C)
- new net: R6.2, U5.9 (B)
- new net: R9.2, U2.5 (K), U2.6 (J)
- new net: R10.2, U2.10 (J), U2.11 (K)
- new net: R11.2, U3.5 (K), U3.6 (J)
- no-connect marks 1 -> 6
Other:
- note added: "555 timer"
- note added: "JK bistabili"
- note added: "LED diode"
- note added: "Montažne rupe"
- note added: "Napajanje"
- note added: "Napajanje bistabila"
- note added: "Reset brojača"
- note added: "Tipkalo i ulaz radnog takta"
- moved on the sheet: C1, C2, C3, D1, D2, D3, D4, D5, J1, L1, R13, R6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

Commit message: vj4-zavrsavanje
Parts:
- removed SW2: ~, symbol Switch:SW_SPDT
- added SW2: SW_Wuerth_450301014042, Button_Switch_THT:SW_Slide-03_Wuerth-WS-SLTV_10x2.5x6.4_P2.54mm, symbol Switch:SW_Wuerth_450301014042
- renumbered R6 to R1, R7 to R2, R8 to R3, R9 to R4, U1 to U6
Connections:
- net 555: now also SW2.2 (C)
- net Clock: now also SW2.1 (B)
- net at C3.2, R13.2: now also SW2.3 (A)
Changed lines of the file:
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@@
 		(dnp no)
 		(fields_autoplaced yes)
-		(property "Reference" "U1"
+		(property "Reference" "U6"
 			(at 160.02 159.9498 0)
 			(effects
@@
 			(project ""
 				(path "/aea8c96d-773b-4621-89b6-2dd77fccfb58"
-					(reference "U1")
+					(reference "U6")
 					(unit 1)
 				)
@@
 	)
 	(symbol
+		(lib_name "Screw_Terminal_01x02_1")
+		(lib_id "Connector:Screw_Terminal_01x02")
+		(at 16.51 44.45 180)
+		(unit 1)
+		(exclude_from_sim no)
+		(in_bom yes)
+		(on_board yes)
+		(dnp no)
+		(property "Reference" "J1"
+			(at 16.51 39.37 0)
+			(effects
+				(font
+					(size 1.27 1.27)
+				)
+			)
+		)
+		(property "Value" "Screw_Terminal_01x02"
+			(at 16.51 38.1 0)
+			(effects
+				(font
+					(size 1.27 1.27)
+				)
+				(hide yes)
+			)
+		)
+		(property "Footprint" ""
+			(at 16.51 44.45 0)
+			(effects
+				(font
+					(size 1.27 1.27)
+				)
+				(hide yes)
+			)
+		)
+		(property "Datasheet" "~"
+			(at 16.51 44.45 0)
+			(effects
+				(font
+					(size 1.27 1.27)
+				)
+				(hide yes)
+			)
+		)
+		(property "Description" "Generic screw terminal, single row, 01x02, script generated (kicad-library-utils/schlib/autogen/connector/)"
+			(at 16.51 44.45 0)
+			(effects
+				(font
+					(size 1.27 1.27)
+				)
+				(hide yes)
+			)
+		)
+		(pin "1"
+		)
+		(pin "2"
+		)
+		(instances
+			(project ""
+				(path "/aea8c96d-773b-4621-89b6-2dd77fccfb58"
+					(reference "J1")
+					(unit 1)
+				)
+			)
+		)
+	)
+	(symbol
 		(lib_id "power:+5V")
 		(at 106.68 24.13 0)
@@
 		(on_board yes)
 		(dnp no)
-		(property "Reference" "R8"
+		(property "Reference" "R3"
 			(at 265.43 39.878 90)
 			(effects
@@
 			(project "PTP_Marko_Pticek_Project1"
 				(path "/aea8c96d-773b-4621-89b6-2dd77fccfb58"
-					(reference "R8")
+					(reference "R3")
 					(unit 1)
 				)
@@
 	)
 	(symbol
-		(lib_id "Connector:Screw_Terminal_01x02")
-		(at 16.51 41.91 0)
-		(mirror y)
-		(unit 1)
-		(exclude_from_sim no)
-		(in_bom yes)
-		(on_board yes)
-		(dnp no)
-		(property "Reference" "J1"
-			(at 16.51 38.862 0)
-			(effects
-				(font
-					(size 1.27 1.27)
-				)
-			)
-		)
-		(property "Value" "Screw_Terminal_01x02"
-			(at 16.51 38.1 0)
-			(effects
-				(font
-					(size 1.27 1.27)
-				)
-				(hide yes)
-			)
-		)
-		(property "Footprint" ""
-			(at 16.51 41.91 0)
-			(effects
-				(font
-					(size 1.27 1.27)
-				)
-				(hide yes)
-			)
-		)
-		(property "Datasheet" "~"
-			(at 16.51 41.91 0)
-			(effects
-				(font
-					(size 1.27 1.27)
-				)
-				(hide yes)
-			)
-		)
-		(property "Description" "Generic screw terminal, single row, 01x02, script generated (kicad-library-utils/schlib/autogen/connector/)"
-			(at 16.51 41.91 0)
-			(effects
-				(font
-					(size 1.27 1.27)
-				)
-				(hide yes)
-			)
-		)
-		(pin "2"
-		)
-		(pin "1"
-		)
-		(instances
-			(project ""
-				(path "/aea8c96d-773b-4621-89b6-2dd77fccfb58"
-					(reference "J1")
-					(unit 1)
-				)
-			)
-		)
-	)
-	(symbol
 		(lib_id "power:GND")
 		(at 226.06 113.03 0)
@@
 		(on_board yes)
 		(dnp no)
-		(property "Reference" "R9"
+		(property "Reference" "R4"
 			(at 265.43 51.308 90)
 			(effects
@@
 			(project "PTP_Marko_Pticek_Project1"
 				(path "/aea8c96d-773b-4621-89b6-2dd77fccfb58"
-					(reference "R9")
+					(reference "R4")
 					(unit 1)
 				)
@@
 		(on_board yes)
 		(dnp no)
-		(property "Reference" "R7"
+		(property "Reference" "R2"
 			(at 265.43 29.718 90)
 			(effects
@@
 			(project "PTP_Marko_Pticek_Project1"
 				(path "/aea8c96d-773b-4621-89b6-2dd77fccfb58"
-					(reference "R7")
+					(reference "R2")
 					(unit 1)
 				)
@@
 	)
 	(symbol
-		(lib_id "Switch:SW_SPDT")
-		(at 58.42 105.41 0)
-		(mirror y)
-		(unit 1)
-		(exclude_from_sim no)
-		(in_bom yes)
-		(on_board yes)
-		(dnp no)
-		(property "Reference" "SW2"
-			(at 58.674 110.744 0)
-			(effects
-				(font
-					(size 1.27 1.27)
-				)
-			)
-		)
-		(property "Value" "~"
-			(at 58.42 99.06 0)
-			(effects
-				(font
-					(size 1.27 1.27)
-				)
-				(hide yes)
-			)
-		)
-		(property "Footprint" ""
-			(at 58.42 105.41 0)
-			(effects
-				(font
-					(size 1.27 1.27)
-				)
-				(hide yes)
-			)
-		)
-		(property "Datasheet" "~"
-			(at 58.42 113.03 0)
-			(effects
-				(font
-					(size 1.27 1.27)
-				)
-				(hide yes)
-			)
-		)
-		(property "Description" "Switch, single pole double throw"
-			(at 58.42 105.41 0)
-			(effects
-				(font
-					(size 1.27 1.27)
-				)
-				(hide yes)
-			)
-		)
-		(pin "3"
-		)
-		(pin "1"
-		)
-		(pin "2"
-		)
-		(instances
-			(project ""
-				(path "/aea8c96d-773b-4621-89b6-2dd77fccfb58"
-					(reference "SW2")
-					(unit 1)
-				)
-			)
-		)
-	)
-	(symbol
 		(lib_id "power:GND")
 		(at 130.81 111.76 0)
@@
 		(on_board yes)
 		(dnp no)
-		(property "Reference" "R6"
+		(property "Reference" "R1"
 			(at 265.43 18.034 90)
 			(effects
@@
 			(project ""
 				(path "/aea8c96d-773b-4621-89b6-2dd77fccfb58"
-					(reference "R6")
+					(reference "R1")
 					(unit 1)
 				)
@@
 				)
 			)
+		)
+	)
+	(symbol
+		(lib_id "Switch:SW_Wuerth_450301014042")
+		(at 58.42 105.41 0)
+		(mirror y)
+		(unit 1)
+		(exclude_from_sim no)
+		(in_bom yes)
+		(on_board yes)
+		(dnp no)
+		(property "Reference" "SW2"
+			(at 58.674 100.33 0)
+			(effects
+				(font
+					(size 1.27 1.27)
+				)
+			)
+		)
+		(property "Value" "SW_Wuerth_450301014042"
+			(at 58.42 99.06 0)
+			(effects
+				(font
+					(size 1.27 1.27)
+				)
+				(hide yes)
+			)
+		)
+		(property "Footprint" "Button_Switch_THT:SW_Slide-03_Wuerth-WS-SLTV_10x2.5x6.4_P2.54mm"
+			(at 58.42 115.57 0)
+			(effects
+				(font
+					(size 1.27 1.27)
+				)
+				(hide yes)
+			)
+		)
+		(property "Datasheet" "https://www.we-online.com/components/products/datasheet/450301014042.pdf"
+			(at 58.42 113.03 0)
+			(effects
+				(font
+					(size 1.27 1.27)
+				)
+				(hide yes)
+			)
+		)
+		(property "Description" "Switch slide, single pole double throw"
+			(at 58.42 105.41 0)
+			(effects
+				(font
+					(size 1.27 1.27)
+				)
+				(hide yes)
+			)
+		)
+		(pin "2"
+		)
+		(pin "1"
+		)
+		(pin "3"
+		)
+		(instances
+			(project ""
+				(path "/aea8c96d-773b-4621-89b6-2dd77fccfb58"
+					(reference "SW2")
+					(unit 1)
+				)
+			)

Commit message: VJ4 - FINAL
Parts:
- removed U5: FYS-3911BUHR-21, Display_7Segment:7SegmentLED_LTS6760_LTS6780, symbol Display_Character:SM420561N
- removed U6: 74LVC1G11, SOT_23_6:SOT-23-6, symbol SN74LVC1G11:SN74LVC1G11
- added U5: HDSP-7401, Display_7Segment:HDSP-7401, symbol Display_Character:HDSP-7401
- added U6: 74LVC1G11, Package_TO_SOT_SMD:SOT-23-6, symbol 74xGxx:74LVC1G11
- D1, D2, D3, D5: footprint (none) -> LED_THT:LED_D5.0mm
- D4: footprint (none) -> Diode_THT:D_DO-41_SOD81_P12.70mm_Horizontal; Manufacturer  (none) -> SMC DIODE SOLUTIONS; Manufacturer Part Number  (none) -> 11DQ06TA
- H1, H2, H3, H4: footprint (none) -> MountingHole:MountingHole_5.5mm
- J1: footprint (none) -> TerminalBlock_MetzConnect:TerminalBlock_MetzConnect_Type011_RT05502HBLC_1x02_P5.00mm_Horizontal; Manufacturer  (none) -> DEGSON ELECTRONICS; Manufacturer Part Number  (none) -> DG301-5.0-02P-12-00A(H)
- L1: footprint (none) -> Inductor_THT:L_Radial_D7.2mm_P3.00mm_Murata_1700; Manufacturer  (none) -> FERROCORE; Manufacturer Part Number  (none) -> COIL0608-0.33
- R1, R2, R3, R4: footprint (none) -> Resistor_THT:R_Axial_DIN0207_L6.3mm_D2.5mm_P10.16mm_Horizontal
- R10, R11, R12, R15, R7, R9: footprint (none) -> Resistor_SMD:R_1206_3216Metric_Pad1.30x1.75mm_HandSolder
- R13: footprint (none) -> Resistor_SMD:R_1206_3216Metric_Pad1.30x1.75mm_HandSolder; Manufacturer  (none) -> ROYALOHM; Manufacturer Part Number (none) -> 1206S4F2001T5E
- R14, R16, R17, R18, R5, R6, R8: footprint (none) -> Resistor_SMD:R_1206_3216Metric_Pad1.30x1.75mm_HandSolder; Manufacturer  (none) -> ROYALOHM; Manufacturer Part Number  (none) -> 1206S4F2001T5E
- R19, R20: footprint (none) -> Resistor_SMD:R_1206_3216Metric_Pad1.30x1.75mm_HandSolder; Manufacturer  (none) -> ROYALOHM; Manufacturer Part Number  (none) -> 1206S4J0473T5E
- SW1: footprint (none) -> Button_Switch_THT:SW_PUSH_6mm_H4.3mm; Manufacturer  (none) -> microswitch TACT; Manufacturer Part Number  (none) -> TACT-64N-F
- SW2: footprint Button_Switch_THT:SW_Slide-03_Wuerth-WS-SLTV_10x2.5x6.4_P2.54mm -> Button_Switch_THT:SW_Slide_SPDT_Straight_CK_OS102011MS2Q; Manufacturer  (none) -> C&K; Manufacturer Part Number  (none) -> OS102011MS2QN1C
- U1: footprint Package_DIP:DIP-8_W7.62mm -> Package_DIP:DIP-8_W7.62mm_Socket_LongPads; Manufacturer  (none) -> ONSEMI; Manufacturer Part Number  (none) -> LM2574N-5G
- U2, U3: footprint (none) -> Package_DIP:DIP-8_W7.62mm_Socket_LongPads; Manufacturer  (none) -> RENESAS; Manufacturer Part Number  (none) -> CD4027BMS
- U4: footprint (none) -> Package_DIP:DIP-16_W7.62mm_Socket_LongPads; Manufacturer  (none) -> TEXAS INSTRUMENTS; Manufacturer Part Number  (none) -> SN74LS47N
- U7: Manufacturer  (none) -> TEXAS INSTRUMENTS; Manufacturer Part Number  (none) -> NE555P
Connections:
- net +5V: now also U5.1 (CA), U5.6 (CA), U6.5 (VCC)
- net Clock: now also U6.3
- net GND: now also U6.2 (GND)
- net Q1: now also U6.6
- net Q3: now also U6.1
- net RESET: now also U6.4
- net at R5.2: now also U5.10 (A)
- net at R17.2: now also U5.2 (F)
- net at R18.2: now also U5.3 (G)
- net at R16.2: now also U5.4 (E)
- net at R14.2: now also U5.5 (D)
- net at R8.2: now also U5.8 (C)
- net at R6.2: now also U5.9 (B)

Commit message: vj7
Parts:
- U2, U3: footprint Package_DIP:DIP-8_W7.62mm_Socket_LongPads -> Package_DIP:DIP-16_W7.62mm_Socket_LongPads
Changed lines of the file:
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@@
 			)
 		)
-		(property "Footprint" "Package_DIP:DIP-8_W7.62mm_Socket_LongPads"
+		(property "Footprint" "Package_DIP:DIP-16_W7.62mm_Socket_LongPads"
 			(at 172.72 104.14 0)
 			(effects
@@
 			)
 		)
-		(property "Footprint" "Package_DIP:DIP-8_W7.62mm_Socket_LongPads"
+		(property "Footprint" "Package_DIP:DIP-16_W7.62mm_Socket_LongPads"
 			(at 110.49 104.14 0)
 			(effects
@@
 			)
 		)
-		(property "Footprint" "Package_DIP:DIP-8_W7.62mm_Socket_LongPads"
+		(property "Footprint" "Package_DIP:DIP-16_W7.62mm_Socket_LongPads"
 			(at 157.48 41.91 0)
 			(effects
@@
 			)
 		)
-		(property "Footprint" "Package_DIP:DIP-8_W7.62mm_Socket_LongPads"
+		(property "Footprint" "Package_DIP:DIP-16_W7.62mm_Socket_LongPads"
 			(at 152.4 104.14 0)
 			(effects
@@
 			)
 		)
-		(property "Footprint" "Package_DIP:DIP-8_W7.62mm_Socket_LongPads"
+		(property "Footprint" "Package_DIP:DIP-16_W7.62mm_Socket_LongPads"
 			(at 182.88 41.91 0)
 			(effects
@@
 			)
 		)
-		(property "Footprint" "Package_DIP:DIP-8_W7.62mm_Socket_LongPads"
+		(property "Footprint" "Package_DIP:DIP-16_W7.62mm_Socket_LongPads"
 			(at 130.81 104.14 0)
 			(effects
