File: PTP_Marko_Pticek_Project1.kicad_pcb (KiCad board)
At the start: 2 copper layers, 45 parts, among them J1 Screw_Terminal_01x02, SW1 SW_Push, SW2 SW_Wuerth_450301014042, U1 LM2574N-5, U2 4027, U3 4027, U4 74LS47, U5 HDSP-7401, U6 74LVC1G11, U7 NE555P

Commit message: vj7
Parts:
- U2, U3: footprint Package_DIP:DIP-8_W7.62mm_Socket_LongPads -> Package_DIP:DIP-16_W7.62mm_Socket_LongPads
- moved U4 23.0 mm to (159.4, 88.6)
- moved R17 22.3 mm to (178.4, 106.1)
- moved R18 22.0 mm to (178.3, 110.2)
- moved L1 21.3 mm to (154.0, 78.5), turned to 90 degrees
- moved C1 17.3 mm to (162.5, 57.8), turned to -90 degrees
- moved C2 14.2 mm to (163.0, 66.8), turned to 90 degrees
- moved R11 14.2 mm to (141.5, 72.5)
- moved U5 14.1 mm to (194.1, 105.9)
- moved R12 14.0 mm to (145.5, 72.5)
- moved U7 10.2 mm to (125.5, 110.2), turned to 180 degrees
- moved R16 9.34 mm to (177.9, 116.7)
- moved R5 8.55 mm to (178.2, 101.8)
- moved U1 8.39 mm to (157.4, 67.5), turned to 180 degrees
- moved C3 8.33 mm to (134.5, 83.2)
- moved R8 8.30 mm to (178.0, 120.1)
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Routing:
- net +5V: track 0.00 -> 181.8 mm, vias 0 -> 2
- net Q3: track 0.00 -> 110.4 mm, vias 0 -> 4
- net Clock: track 0.00 -> 71.5 mm
- net Q1: track 0.00 -> 68.1 mm, vias 0 -> 4
- net Q2: track 0.00 -> 59.0 mm
- net Q0: track 0.00 -> 58.9 mm
- net RESET: track 0.00 -> 54.4 mm, vias 0 -> 4
- net Net-(D4-K): track 0.00 -> 36.1 mm, vias 0 -> 3
- net Net-(U2A-J): track 0.00 -> 36.0 mm
- net Net-(U4-BI): track 0.00 -> 35.8 mm, vias 0 -> 4
- net 555: track 0.00 -> 31.1 mm
- net VD: track 0.00 -> 31.0 mm
- net Net-(U7-THR): track 0.00 -> 30.4 mm
- net Net-(U4-f): track 0.00 -> 27.1 mm, vias 0 -> 6
- net Net-(U4-c): track 0.00 -> 25.9 mm, vias 0 -> 4
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- added copper zone on B.Cu, net GND

Commit message: dovrsavanje
Parts:
- moved R7 63.5 mm to (161.2, 113.5), turned to 90 degrees
- moved SW1 57.9 mm to (162.2, 121.3)
- moved R15 57.3 mm to (189.2, 87.1)
- moved R13 56.3 mm to (158.4, 113.5), turned to 90 degrees
- moved R11 49.6 mm to (169.4, 113.5)
- moved R9 48.8 mm to (164.0, 113.5)
- moved R12 48.8 mm to (172.0, 113.5)
- moved R10 45.9 mm to (166.8, 113.5)
- moved D4 41.7 mm to (131.5, 59.4), turned to 0 degrees
- moved C1 37.0 mm to (125.8, 62.6), turned to 90 degrees
- moved C3 36.7 mm to (155.4, 113.4), turned to 90 degrees
- moved R1 35.9 mm to (187.2, 60.3), turned to -90 degrees
- moved R4 34.2 mm to (159.8, 59.9), turned to -90 degrees
- moved U6 33.7 mm to (139.1, 95.8)
- moved R2 30.4 mm to (179.0, 60.1), turned to -90 degrees
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Routing:
- net Q0: track 58.9 -> 141.3 mm, vias 0 -> 1
- net +5V: track 181.8 -> 248.3 mm, vias 2 -> 1
- net GND: track 0.00 -> 56.9 mm, vias 0 -> 2
- net Net-(U3A-J): track 5.42 -> 32.9 mm, vias 2 -> 0
- net Q3: track 110.4 -> 87.7 mm
- net Q2: track 59.0 -> 37.7 mm, vias 0 -> 2
- net Net-(U4-f): track 27.1 -> 7.42 mm, vias 6 -> 1
- net Net-(U4-g): track 23.6 -> 5.28 mm, vias 4 -> 0
- net RESET: track 54.4 -> 36.5 mm, vias 4 -> 1
- net Q1: track 68.1 -> 50.5 mm, vias 4 -> 1
- net (no net): track 16.8 -> 0.00 mm, vias 4 -> 0
- net Net-(U3B-J): track 2.54 -> 19.0 mm
- net Net-(U4-BI): track 35.8 -> 19.9 mm, vias 4 -> 0
- net Net-(SW2-A): track 25.0 -> 40.3 mm, vias 2 -> 0
- net Net-(U2B-J): track 2.54 -> 17.4 mm
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Other:
- board outline added: 100 x 80 mm
